Commit message: 周期性输出调制解调传感器数据

File: src/eca_a9/eca_a9_description/urdf/eca_a9_base.xacro (robot description, xacro)
@@ -28,4 +28,6 @@
   <xacro:property name="area" value="0.04155"/>
   <xacro:property name="length" value="1.98"/>
+  <!-- Global RPT auto repeat period (seconds) for reuse -->
+  <xacro:property name="rpt_auto_repeat_period" value="5.0"/>
   <xacro:property name="visual_mesh_file" value="file://$(find eca_a9_description)/mesh/eca_a9.dae"/>
   <xacro:property name="collision_mesh_file" value="file://$(find eca_a9_description)/mesh/eca_a9.stl"/>

File: src/eca_a9/eca_a9_description/urdf/eca_a9_sensors.xacro (robot description, xacro)
@@ -68,5 +68,6 @@
         subscribe_enabled="true"
         processing_enabled="true"
-        default_target_ns="eca_a9_2">
+        default_target_ns="eca_a9_2"
+        auto_repeat_period="${rpt_auto_repeat_period}">
         <origin xyz="0 0 0" rpy="0 0 0"/>
       </xacro:default_rpt>

File: src/uuv_simulator-noetic/uuv_sensor_plugins/uuv_sensor_ros_plugins/urdf/rpt_snippets.xacro (robot description, xacro)
@@ -21,5 +21,5 @@
     </collision>
   </xacro:macro>
-  <xacro:macro name="default_rpt" params="namespace parent_link *origin sound_speed:=1500.0 max_range:=12000.0 advertise_enabled:=false subscribe_enabled:=false processing_enabled:=false default_target_ns:=''"><!-- default_target_ns empty string by default -->
+  <xacro:macro name="default_rpt" params="namespace parent_link *origin update_rate:=0.2 sound_speed:=1500.0 max_range:=12000.0 advertise_enabled:=false subscribe_enabled:=false processing_enabled:=false default_target_ns:='' auto_repeat_period:=0.0"><!-- default_target_ns empty string by default -->
     <xacro:rpt_plugin_macro
       namespace="${namespace}"
@@ -29,4 +29,5 @@
       noise_sigma="0.0"
       topic="rpt"
+      update_rate="${update_rate}"
       sound_speed="${sound_speed}"
       max_range="${max_range}"
@@ -34,10 +35,11 @@
       subscribe_enabled="${subscribe_enabled}"
       processing_enabled="${processing_enabled}"
-      default_target_ns="${default_target_ns}">
+      default_target_ns="${default_target_ns}"
+      auto_repeat_period="${auto_repeat_period}">
       <xacro:insert_block name="origin" />
     </xacro:rpt_plugin_macro>
   </xacro:macro>
   <xacro:macro name="rpt_plugin_macro"
-    params="namespace suffix parent_link topic noise_sigma noise_amplitude sound_speed:=1500.0 max_range:=12000.0 advertise_enabled:=false subscribe_enabled:=false processing_enabled:=false default_target_ns:='' *origin">
+    params="namespace suffix parent_link topic noise_sigma noise_amplitude update_rate:=0.2 sound_speed:=1500.0 max_range:=12000.0 advertise_enabled:=false subscribe_enabled:=false processing_enabled:=false default_target_ns:='' auto_repeat_period:=0.0 *origin">
     <link name="${namespace}/rpt${suffix}_link">
       <inertial>
@@ -66,5 +68,5 @@
         <static_reference_frame>world</static_reference_frame> <!-- name of the reference frame of all position measurements -->
         <sensor_topic>${topic}</sensor_topic> <!-- name of the sensor output topic and prefix of service name -->
-        <update_rate>30</update_rate>
+        <update_rate>${update_rate}</update_rate>
         <noise_sigma>${noise_sigma}</noise_sigma> <!-- std dev of position estimates in x, y, z [m] -->
         <noise_amplitude>${noise_amplitude}</noise_amplitude>
