Commit message: 09081806

File: src/eca_a9/eca_a9_description/urdf/eca_a9_sensors.xacro (robot description, xacro)
@@ -27,5 +27,5 @@
       noise_sigma="0"
       noise_amplitude="0"
-      update_rate="7"
+      update_rate="20"
       reference_frame="world">
       <origin xyz="0.4785 0.0 -0.0825" rpy="0 ${0.5*pi} 0" />
@@ -72,8 +72,26 @@
       power_load="5"
       topic="${namespace}/pressure/state"/>
-    <!-- IMU  -->
-    <xacro:default_imu namespace="${namespace}" parent_link="${namespace}/base_link">
+    <!-- IMU (navigation-grade override) -->
+    <xacro:imu_plugin_macro
+      namespace="${namespace}"
+      imu_suffix=""
+      parent_link="${namespace}/base_link"
+      imu_topic="imu"
+      mass_imu_sensor="0.015"
+      gyroscope_noise_density="0.000003"
+      gyroscope_random_walk="0.0000003"
+      gyroscope_bias_correlation_time="3600.0"
+      gyroscope_turn_on_bias_sigma="0.0020"
+      accelerometer_noise_density="0.00003"
+      accelerometer_random_walk="0.000050"
+      accelerometer_bias_correlation_time="3600.0"
+      accelerometer_turn_on_bias_sigma="0.0500"
+      orientation_noise="0.002"
+      enable_local_ned_frame="false"
+      reference_frame="world"
+      update_rate="200">
+      <inertia ixx="0.00001" ixy="0.0" ixz="0.0" iyy="0.00001" iyz="0.0" izz="0.00001" />
       <origin xyz="0 0 0" rpy="0 0 0"/>
-    </xacro:default_imu>
+    </xacro:imu_plugin_macro>
     <xacro:switchable_battery_consumer_macro
       link_name="${namespace}/imu_link"

Commit message: 20250911初步加入声学调制解调器

File: src/eca_a9/eca_a9_description/urdf/eca_a9_sensors.xacro (robot description, xacro)
@@ -58,8 +58,18 @@
       power_load="25"
       topic="${namespace}/sonarright/state"/>
-    <!-- RPT
-    <xacro:default_rpt namespace="${namespace}" parent_link="${namespace}/base_link">
-      <origin xyz="0 0 0" rpy="0 0 0"/>
-    </xacro:default_rpt>  -->
+    <!-- RPT: enable TWTT only for eca_a9_1 targeting eca_a9_2 -->
+    <xacro:if value="${namespace == 'eca_a9_1'}">
+      <xacro:default_rpt
+        namespace="${namespace}"
+        parent_link="${namespace}/base_link"
+        sound_speed="1500.0"
+        max_range="12000.0"
+        advertise_enabled="true"
+        subscribe_enabled="true"
+        processing_enabled="true"
+        default_target_ns="eca_a9_2">
+        <origin xyz="0 0 0" rpy="0 0 0"/>
+      </xacro:default_rpt>
+    </xacro:if>
     <!-- Pressure -->
     <xacro:default_pressure namespace="${namespace}" parent_link="${namespace}/base_link">
@@ -134,3 +144,4 @@
       <origin xyz="0 0 0" rpy="0 0 0"/>
     </xacro:default_chemical_concentration_sensor>
+    <!-- Acoustic modem (removed) -->
 </robot>

File: src/uuv_simulator-noetic/uuv_sensor_plugins/uuv_sensor_ros_plugins/urdf/chemical_concentration_snippets.xacro (robot description, xacro)
@@ -115,4 +115,5 @@
        <noise_sigma>${noise_sigma}</noise_sigma>
        <noise_amplitude>${noise_amplitude}</noise_amplitude>
+       <is_on>true</is_on>
      </plugin>
    </gazebo>

File: src/uuv_simulator-noetic/uuv_sensor_plugins/uuv_sensor_ros_plugins/urdf/rpt_snippets.xacro (robot description, xacro)
@@ -21,5 +21,5 @@
     </collision>
   </xacro:macro>
-  <xacro:macro name="default_rpt" params="namespace parent_link *origin">
+  <xacro:macro name="default_rpt" params="namespace parent_link *origin sound_speed:=1500.0 max_range:=12000.0 advertise_enabled:=false subscribe_enabled:=false processing_enabled:=false default_target_ns:=''"><!-- default_target_ns empty string by default -->
     <xacro:rpt_plugin_macro
       namespace="${namespace}"
@@ -28,11 +28,16 @@
       noise_amplitude="0.0"
       noise_sigma="0.0"
-      topic="rpt">
+      topic="rpt"
+      sound_speed="${sound_speed}"
+      max_range="${max_range}"
+      advertise_enabled="${advertise_enabled}"
+      subscribe_enabled="${subscribe_enabled}"
+      processing_enabled="${processing_enabled}"
+      default_target_ns="${default_target_ns}">
       <xacro:insert_block name="origin" />
     </xacro:rpt_plugin_macro>
   </xacro:macro>
   <xacro:macro name="rpt_plugin_macro"
-    params="namespace suffix parent_link topic noise_sigma noise_amplitude
-    *origin">
+    params="namespace suffix parent_link topic noise_sigma noise_amplitude sound_speed:=1500.0 max_range:=12000.0 advertise_enabled:=false subscribe_enabled:=false processing_enabled:=false default_target_ns:='' *origin">
     <link name="${namespace}/rpt${suffix}_link">
       <inertial>
@@ -59,10 +64,17 @@
         <robot_namespace>${namespace}</robot_namespace> <!-- ros namespace in which the messages are published -->
         <link_name>${namespace}/rpt${suffix}_link</link_name> <!-- sensor link name -->
-        <static_reference_frame>ssbl</static_reference_frame> <!-- name of the refernce frame of all position measurements -->
+        <static_reference_frame>world</static_reference_frame> <!-- name of the reference frame of all position measurements -->
         <sensor_topic>${topic}</sensor_topic> <!-- name of the sensor output topic and prefix of service name -->
-        <update_rate>0.5</update_rate> <!-- Update period [s] -->
+        <update_rate>30</update_rate>
         <noise_sigma>${noise_sigma}</noise_sigma> <!-- std dev of position estimates in x, y, z [m] -->
         <noise_amplitude>${noise_amplitude}</noise_amplitude>
         <enable_gazebo_messages>false</enable_gazebo_messages>
+        <!-- Optional TWTT acoustic extension parameters -->
+        <sound_speed>${sound_speed}</sound_speed>
+        <max_range>${max_range}</max_range>
+        <advertise_enabled>${advertise_enabled}</advertise_enabled>
+        <subscribe_enabled>${subscribe_enabled}</subscribe_enabled>
+        <processing_enabled>${processing_enabled}</processing_enabled>
+        <default_target_ns>${default_target_ns}</default_target_ns>
       </plugin>
     </gazebo>

Commit message: 20250922

File: src/eca_a9/eca_a9_description/urdf/eca_a9_sensors.xacro (robot description, xacro)
@@ -58,19 +58,17 @@
       power_load="25"
       topic="${namespace}/sonarright/state"/>
-    <!-- RPT: enable TWTT only for eca_a9_1 targeting eca_a9_2 -->
-    <xacro:if value="${namespace == 'eca_a9_1'}">
-      <xacro:default_rpt
-        namespace="${namespace}"
-        parent_link="${namespace}/base_link"
-        sound_speed="1500.0"
-        max_range="12000.0"
-        advertise_enabled="true"
-        subscribe_enabled="true"
-        processing_enabled="true"
-        default_target_ns="eca_a9_surface"
-        auto_repeat_period="${rpt_auto_repeat_period}">
-        <origin xyz="0 0 0" rpy="0 0 0"/>
-      </xacro:default_rpt>
-    </xacro:if>
+    <!-- RPT: enable OWTT for all vehicles; subscribe to per-vehicle router -->
+    <xacro:default_rpt
+      namespace="${namespace}"
+      parent_link="${namespace}/base_link"
+      sound_speed="1500.0"
+      max_range="12000.0"
+      advertise_enabled="true"
+      subscribe_enabled="true"
+      processing_enabled="true"
+      default_target_ns="router_${namespace}"
+      auto_repeat_period="${rpt_auto_repeat_period}">
+      <origin xyz="0 0 0" rpy="0 0 0"/>
+    </xacro:default_rpt>
     <!-- Pressure -->
     <xacro:default_pressure namespace="${namespace}" parent_link="${namespace}/base_link">

Commit message: DVL深度计互测距加误差噪声一分钟测距周期

File: src/eca_a9/eca_a9_description/urdf/eca_a9_sensors.xacro (robot description, xacro)
@@ -1,3 +1,3 @@
-<?xml version="1.0"?>
+<?xml version="1.0" encoding="UTF-8"?>
 <!-- Copyright (c) 2016 The UUV Simulator Authors.
      All rights reserved.
@@ -28,5 +28,6 @@
       noise_amplitude="0"
       update_rate="20"
-      reference_frame="world">
+      reference_frame="world"
+      relative_velocity_three_sigma="0.1">
       <origin xyz="0.4785 0.0 -0.0825" rpy="0 ${0.5*pi} 0" />
     </xacro:dvl_plugin_macro>
@@ -38,4 +39,5 @@
       topic="${namespace}/dvl/state"/>
     <!-- Side scan sonar left -->
+    <xacro:if value="${0}">
     <xacro:sidescan_sonar namespace="${namespace}" parent_link="${namespace}/base_link" suffix="left">
       <origin xyz="0.41225 0.1498 -0.04615" rpy="${0.5*pi} ${-5*d2r+pi/3.0} ${0.5*pi}" />
@@ -47,5 +49,7 @@
       power_load="25"
       topic="${namespace}/sonarleft/state"/>
+    </xacro:if>
     <!-- Side scan sonar right -->
+    <xacro:if value="${0}">
     <xacro:sidescan_sonar
       namespace="${namespace}" parent_link="${namespace}/base_link" suffix="right">
@@ -58,4 +62,5 @@
       power_load="25"
       topic="${namespace}/sonarright/state"/>
+    </xacro:if>
     <!-- RPT: enable OWTT for all vehicles; subscribe to per-vehicle router -->
     <xacro:default_rpt
@@ -63,14 +68,25 @@
       parent_link="${namespace}/base_link"
       sound_speed="1500.0"
-      max_range="12000.0"
+      max_range="120000.0"
       advertise_enabled="true"
       subscribe_enabled="true"
       processing_enabled="true"
       default_target_ns="router_${namespace}"
-      auto_repeat_period="${rpt_auto_repeat_period}">
+      auto_repeat_period="${rpt_auto_repeat_period}"
+      range_noise_sigma_ratio="0.001"
+      range_noise_sigma_min="0.0"
+      range_noise_additive="true"
+      range_noise_clip_ratio="0.003"> <!-- clip at +/- 0.3% of true range -->
       <origin xyz="0 0 0" rpy="0 0 0"/>
     </xacro:default_rpt>
-    <!-- Pressure -->
-    <xacro:default_pressure namespace="${namespace}" parent_link="${namespace}/base_link">
+    <!-- Pressure: configure for +/- 1 m depth accuracy (3 sigma) -->
+    <!-- With kPaPerM=9.80638 kPa/m, 1 m depth corresponds to 9.80638 kPa change.
+         Set noise_sigma so that 3 sigma ~= 9.80638 kPa => sigma ~= 3.268793 kPa.
+         Use zero-mean white noise: noise_amplitude=1.0 scales the Gaussian draw. -->
+    <xacro:default_pressure
+      namespace="${namespace}"
+      parent_link="${namespace}/base_link"
+      noise_sigma="3.268793"
+      noise_amplitude="1.0">
       <origin xyz="0 0 0" rpy="0 0 0"/>
     </xacro:default_pressure>
@@ -81,5 +97,5 @@
       power_load="5"
       topic="${namespace}/pressure/state"/>
-    <!-- IMU (陀螺常值零偏严格0.001°/h高精度惯导) -->
+    <!-- IMU (high-precision INS, gyro bias 0.001 deg/h) -->
     <xacro:imu_plugin_macro
       namespace="${namespace}"
@@ -110,4 +126,5 @@
       topic="${namespace}/imu/state"/>
     <!-- Mount a camera -->
+    <xacro:if value="${0}">
     <xacro:regular_camera_plugin_macro
         namespace="${namespace}"
@@ -131,5 +148,7 @@
       power_load="25"
       topic=""/>
+    </xacro:if>
     <!-- Mount a GPS. -->
+    <xacro:if value="${0}">
     <xacro:default_gps namespace="${namespace}" parent_link="${namespace}/base_link" />
     <xacro:switchable_battery_consumer_macro
@@ -139,8 +158,11 @@
       power_load="5"
       topic=""/>
+    </xacro:if>
     <!-- Mount the chemical concentration sensor -->
+    <xacro:if value="${0}">
     <xacro:default_chemical_concentration_sensor namespace="${namespace}" parent_link="${namespace}/base_link">
       <origin xyz="0 0 0" rpy="0 0 0"/>
     </xacro:default_chemical_concentration_sensor>
+    </xacro:if>
     <!-- Acoustic modem (removed) -->
 </robot>

File: src/uuv_simulator-noetic/uuv_sensor_plugins/uuv_sensor_ros_plugins/urdf/dvl_snippets.xacro (robot description, xacro)
@@ -31,4 +31,5 @@
       noise_sigma="0"
       noise_amplitude="0"
+      relative_velocity_three_sigma="0.1"
       scale="1">
       <xacro:insert_block name="origin" />
@@ -62,4 +63,5 @@
       noise_sigma="0"
       noise_amplitude="0"
+      relative_velocity_three_sigma="0.1"
       scale="1">
       <xacro:insert_block name="origin" />
@@ -122,5 +124,5 @@
   <xacro:macro name="dvl_plugin_macro"
     params="namespace suffix parent_link topic scale *origin update_rate
-    reference_frame noise_sigma noise_amplitude">
+    reference_frame noise_sigma noise_amplitude relative_velocity_three_sigma">
     <link name="${namespace}/dvl${suffix}_link">
       <inertial>
@@ -167,4 +169,5 @@
         <noise_sigma>${noise_sigma}</noise_sigma> <!-- std dev of position estimates in x, y, z [m/s] -->
         <noise_amplitude>${noise_amplitude}</noise_amplitude>
+        <relative_velocity_three_sigma>${relative_velocity_three_sigma}</relative_velocity_three_sigma>
         <enable_gazebo_messages>false</enable_gazebo_messages>
         <enable_local_ned_frame>false</enable_local_ned_frame>

File: src/uuv_simulator-noetic/uuv_sensor_plugins/uuv_sensor_ros_plugins/urdf/pressure_snippets.xacro (robot description, xacro)
@@ -39,5 +39,5 @@
     </xacro:pressure_plugin_macro>
   </xacro:macro>
-  <xacro:macro name="default_pressure" params="namespace parent_link *origin">
+  <xacro:macro name="default_pressure" params="namespace parent_link *origin update_rate:=10 range:=30000 noise_sigma:=3.0 noise_amplitude:=0.0 estimateDepth:=false standardPressure:=101.325 kPaPerM:=9.80638">
     <xacro:pressure_plugin_macro
       namespace="${namespace}"
@@ -46,11 +46,11 @@
       topic="pressure"
       mass="0.015"
-      update_rate="10"
-      range="30000"
-      noise_sigma="3.0"
-      noise_amplitude="0.0"
-      estimateDepth="false"
-      standardPressure="101.325"
-      kPaPerM="9.80638">
+      update_rate="${update_rate}"
+      range="${range}"
+      noise_sigma="${noise_sigma}"
+      noise_amplitude="${noise_amplitude}"
+      estimateDepth="${estimateDepth}"
+      standardPressure="${standardPressure}"
+      kPaPerM="${kPaPerM}">
       <inertia ixx="0.00001" ixy="0.0" ixz="0.0" iyy="0.00001" iyz="0.0" izz="0.00001" />
       <xacro:insert_block name="origin" />

File: src/uuv_simulator-noetic/uuv_sensor_plugins/uuv_sensor_ros_plugins/urdf/rpt_snippets.xacro (robot description, xacro)
@@ -21,5 +21,5 @@
     </collision>
   </xacro:macro>
-  <xacro:macro name="default_rpt" params="namespace parent_link *origin update_rate:=0.2 sound_speed:=1500.0 max_range:=12000.0 advertise_enabled:=false subscribe_enabled:=false processing_enabled:=false default_target_ns:='' auto_repeat_period:=0.0"><!-- default_target_ns empty string by default -->
+  <xacro:macro name="default_rpt" params="namespace parent_link *origin update_rate:=0.2 sound_speed:=1500.0 max_range:=12000.0 advertise_enabled:=false subscribe_enabled:=false processing_enabled:=false default_target_ns:='' auto_repeat_period:=0.0 range_noise_sigma:=0.0 range_noise_sigma_ratio:=0.0 range_noise_sigma_min:=0.0 range_noise_additive:=true range_noise_clip_ratio:=0.0"><!-- default_target_ns empty string by default -->
     <xacro:rpt_plugin_macro
       namespace="${namespace}"
@@ -36,10 +36,15 @@
       processing_enabled="${processing_enabled}"
       default_target_ns="${default_target_ns}"
-      auto_repeat_period="${auto_repeat_period}">
+      auto_repeat_period="${auto_repeat_period}"
+      range_noise_sigma="${range_noise_sigma}"
+      range_noise_sigma_ratio="${range_noise_sigma_ratio}"
+      range_noise_sigma_min="${range_noise_sigma_min}"
+      range_noise_additive="${range_noise_additive}"
+      range_noise_clip_ratio="${range_noise_clip_ratio}">
       <xacro:insert_block name="origin" />
     </xacro:rpt_plugin_macro>
   </xacro:macro>
   <xacro:macro name="rpt_plugin_macro"
-    params="namespace suffix parent_link topic noise_sigma noise_amplitude update_rate:=0.2 sound_speed:=1500.0 max_range:=12000.0 advertise_enabled:=false subscribe_enabled:=false processing_enabled:=false default_target_ns:='' auto_repeat_period:=0.0 *origin">
+    params="namespace suffix parent_link topic noise_sigma noise_amplitude update_rate:=0.2 sound_speed:=1500.0 max_range:=12000.0 advertise_enabled:=false subscribe_enabled:=false processing_enabled:=false default_target_ns:='' auto_repeat_period:=0.0 range_noise_sigma:=0.0 range_noise_sigma_ratio:=0.0 range_noise_sigma_min:=0.0 range_noise_additive:=true range_noise_clip_ratio:=0.0 *origin">
     <link name="${namespace}/rpt${suffix}_link">
       <inertial>
@@ -79,4 +84,10 @@
         <processing_enabled>${processing_enabled}</processing_enabled>
         <default_target_ns>${default_target_ns}</default_target_ns>
+        <!-- Proportional OWTT range noise (sigma and optional clipping) -->
+        <range_noise_sigma>${range_noise_sigma}</range_noise_sigma>
+        <range_noise_sigma_ratio>${range_noise_sigma_ratio}</range_noise_sigma_ratio>
+        <range_noise_sigma_min>${range_noise_sigma_min}</range_noise_sigma_min>
+        <range_noise_additive>${range_noise_additive}</range_noise_additive>
+        <range_noise_clip_ratio>${range_noise_clip_ratio}</range_noise_clip_ratio>
       </plugin>
     </gazebo>

Commit message: MBES+PF地形匹配导航

File: src/eca_a9/eca_a9_description/urdf/eca_a9_sensors.xacro (robot description, xacro)
@@ -39,5 +39,5 @@
       topic="${namespace}/dvl/state"/>
     <!-- Side scan sonar left -->
-    <xacro:if value="${0}">
+    <xacro:if value="${1}">
     <xacro:sidescan_sonar namespace="${namespace}" parent_link="${namespace}/base_link" suffix="left">
       <origin xyz="0.41225 0.1498 -0.04615" rpy="${0.5*pi} ${-5*d2r+pi/3.0} ${0.5*pi}" />
@@ -51,5 +51,5 @@
     </xacro:if>
     <!-- Side scan sonar right -->
-    <xacro:if value="${0}">
+    <xacro:if value="${1}">
     <xacro:sidescan_sonar
       namespace="${namespace}" parent_link="${namespace}/base_link" suffix="right">
@@ -127,5 +127,5 @@
       topic="${namespace}/imu/state"/>
     <!-- Mount a camera -->
-    <xacro:if value="${0}">
+    <xacro:if value="${1}">
     <xacro:regular_camera_plugin_macro
         namespace="${namespace}"
@@ -166,4 +166,75 @@
     </xacro:default_chemical_concentration_sensor>
     </xacro:if>
+    <!-- Custom Down-Looking MBES (100m range) -->
+  <xacro:macro name="no_collision">
+    <collision>
+      <geometry>
+        <cylinder length="${0.000001}" radius="${0.000001}" />
+      </geometry>
+      <origin xyz="0 0 0" rpy="0 ${0.5*pi} 0"/>
+    </collision>
+  </xacro:macro>
+  <xacro:property name="mbes_suffix" value="_mbes"/>
+  <xacro:property name="mbes_topic" value="mbes"/>
+  <xacro:property name="mbes_fov" value="2.09"/>
+  <xacro:property name="mbes_width" value="512"/>
+  <xacro:property name="mbes_height" value="512"/>
+  <xacro:property name="mbes_update_rate" value="10"/>
+  <xacro:property name="mbes_range_near" value="0.5"/>
+  <xacro:property name="mbes_range_far" value="100.0"/>
+  <!-- MBES Sensor Link -->
+  <link name="${namespace}/forward_sonar${mbes_suffix}_link">
+    <inertial>
+      <inertia ixx="0.00001" ixy="0.0" ixz="0.0" iyy="0.00001" iyz="0.0" izz="0.00001" />
+      <mass value="0.015" />
+      <origin xyz="0 0 0" rpy="0 0 0" />
+    </inertial>
+    <visual>
+      <geometry>
+        <box size="0.05 0.05 0.02"/>
+      </geometry>
+    </visual>
+    <xacro:no_collision/>
+  </link>
+  <joint name="${namespace}_forward_sonar${mbes_suffix}_joint" type="fixed">
+    <!-- Mounted at bottom, looking DOWN (Pitch = pi/2) -->
+    <origin xyz="0.6 0 -0.12" rpy="0 1.5708 0"/>
+    <parent link="${namespace}/base_link" />
+    <child link="${namespace}/forward_sonar${mbes_suffix}_link" />
+  </joint>
+  <gazebo reference="${namespace}/forward_sonar${mbes_suffix}_link">
+    <sensor name="${namespace}/image_sonar" type="depth">
+      <camera>
+        <horizontal_fov>${mbes_fov}</horizontal_fov>
+        <image>
+          <width>${mbes_width}</width>
+          <height>${mbes_height}</height>
+          <format>R8G8B8</format>
+        </image>
+        <clip>
+          <near>${mbes_range_near}</near>
+          <far>${mbes_range_far}</far>
+        </clip>
+      </camera>
+      <plugin filename="libgazebo_ros_depth_camera.so" name="forward_sonar${mbes_suffix}_controller">
+        <cameraName>depth</cameraName>
+        <imageTopicName>image_raw_color</imageTopicName>
+        <cameraInfoTopicName>camera_info_color</cameraInfoTopicName>
+        <depthImageTopicName>image_raw</depthImageTopicName>
+        <depthImageCameraInfoTopicName>camera_info</depthImageCameraInfoTopicName>
+        <pointCloudTopicName>points</pointCloudTopicName>
+        <frameName>${namespace}/forward_sonar${mbes_suffix}_optical_frame</frameName>
+        <updateRate>${mbes_update_rate}</updateRate>
+      </plugin>
+      <always_on>true</always_on>
+      <update_rate>${mbes_update_rate}</update_rate>
+    </sensor>
+  </gazebo>
+  <joint name="${namespace}/forward_sonar${mbes_suffix}_joint" type="fixed">
+    <origin xyz="0 0 0" rpy="${-pi/2} 0 ${-pi/2}"/>
+    <parent link="${namespace}/forward_sonar${mbes_suffix}_link"/>
+    <child link="${namespace}/forward_sonar${mbes_suffix}_optical_frame"/>
+  </joint>
+  <link name="${namespace}/forward_sonar${mbes_suffix}_optical_frame"/>
     <!-- Acoustic modem (removed) -->
 </robot>

Commit message: 相对高度匹配

File: src/eca_a9/eca_a9_description/urdf/eca_a9_sensors.xacro (robot description, xacro)
@@ -177,7 +177,7 @@
   <xacro:property name="mbes_suffix" value="_mbes"/>
   <xacro:property name="mbes_topic" value="mbes"/>
-  <xacro:property name="mbes_fov" value="2.09"/>
-  <xacro:property name="mbes_width" value="512"/>
-  <xacro:property name="mbes_height" value="512"/>
+  <xacro:property name="mbes_fov" value="1.047"/>
+  <xacro:property name="mbes_width" value="64"/>
+  <xacro:property name="mbes_height" value="64"/>
   <xacro:property name="mbes_update_rate" value="10"/>
   <xacro:property name="mbes_range_near" value="0.5"/>
