Commit message: 模型加入科里奥利力并补偿-仿真加速

File: src/eca_a9/eca_a9_description/robots/eca_a9_default.urdf.xacro (robot description, xacro)
@@ -16,4 +16,6 @@
   <xacro:arg name="namespace" default="eca_a9"/>
   <xacro:arg name="inertial_reference_frame" default="world"/>
+  <!-- Mission latitude in radians for Earth Coriolis force calculation -->
+  <xacro:arg name="mission_latitude" default="0.3183"/>  <!-- 18.25 degrees North (Sanya) by default -->
   <!-- Include the UUV macro file -->
   <xacro:include filename="$(find eca_a9_description)/urdf/eca_a9_base.xacro"/>
@@ -22,4 +24,5 @@
     namespace="$(arg namespace)"
     debug="$(arg debug)"
+    mission_latitude="$(arg mission_latitude)"
     inertial_reference_frame="$(arg inertial_reference_frame)"/>
   <!-- Joint state publisher plugin -->

File: src/eca_a9/eca_a9_description/urdf/eca_a9_base.xacro (robot description, xacro)
@@ -34,5 +34,5 @@
   <xacro:property name="prop_mesh_file" value="file://$(find eca_a9_description)/mesh/eca_a9_propeller.dae"/>
   <xacro:property name="fin_mesh_file" value="file://$(find eca_a9_description)/mesh/eca_a9_fin.dae"/>
-  <xacro:macro name="eca_a9_base" params="namespace debug inertial_reference_frame">
+  <xacro:macro name="eca_a9_base" params="namespace debug inertial_reference_frame mission_latitude:=0.3183">
     <link name="${namespace}/base_link">
       <visual>
@@ -68,4 +68,9 @@
           <hydrodynamic_model>
             <type>fossen</type>
+            <!-- Enable Earth rotation Coriolis force for long-duration navigation (170 hours) -->
+            <enable_earth_coriolis>true</enable_earth_coriolis>
+            <!-- Vehicle latitude in radians (passed from launch parameters) -->
+            <!-- This should be set based on your actual mission area -->
+            <vehicle_latitude>${mission_latitude}</vehicle_latitude>
             <added_mass>
               4   0   0   0   0   0
