Commit message: 精简版

File: src/uuv_simulator-noetic/uuv_descriptions/robots/rexrov_sonar.xacro (robot description, xacro)
@@ -35,7 +35,18 @@
     </gazebo>
   </xacro:rexrov_base>
-  <xacro:forward_multibeam_sonar_m450_130 namespace="$(arg namespace)" parent_link="$(arg namespace)/base_link">
+  <xacro:forward_looking_sonar
+    namespace="$(arg namespace)"
+    suffix=""
+    parent_link="$(arg namespace)/base_link"
+    topic="sonar"
+    mass="0.015"
+    update_rate="25"
+    samples="768"
+    fov="2.27"
+    width="768"
+    height="492">
+    <inertia ixx="0.00001" ixy="0.0" ixz="0.0" iyy="0.00001" iyz="0.0" izz="0.00001" />
     <origin xyz="1.4 0 0.65" rpy="0 0 0"/>
-  </xacro:forward_multibeam_sonar_m450_130>
+  </xacro:forward_looking_sonar>
   <!-- Joint state publisher plugin -->
   <xacro:default_joint_state_publisher namespace="$(arg namespace)" update_rate="50"/>

File: src/uuv_simulator-noetic/uuv_sensor_plugins/uuv_sensor_ros_plugins/urdf/sonar_snippets.xacro (robot description, xacro)
@@ -187,5 +187,5 @@
           <clip>
             <near>0.1</near>
-            <far>17</far>
+            <far>150</far>
           </clip>
           <save enabled="true">
